Commit message: Close the six scored gaps from the watched flight
Spec: .scratch/mission2-final-gaps/spec.md. Evidence: VERIFICATION.md §13.
Offline suite 735 passed, 3 skipped (skips are the deferred photo corpus).

Restricted zones (10 marks, -5 per violation). §12.3 retracted "red zones are
never detected" and left a narrow question: 198 exclusions confirmed and the
aircraft still overflew red ground. The answer was scope -- only sweep LANES
were clipped, and every straight leg flew mav.goto() untouched, including the
transit between two clipped lane segments. Adds route_leg/merge_exclusions/
leg_hits_exclusion/point_in_exclusion to the search planner and a shared
LegRouter; Goto, GotoHome, ReturnToCorridorMouth, DescendToDecode and
LawnmowerSearch route, ApproachBanner checks and aborts (a visual servo cannot
detour without losing the lock). A blocked leg is always an abort with a
reason; the straight line is never the fallback.

Banner sweep. Replaces the continuous yaw with STEP/SETTLE/DWELL/DECIDE/CENTRE
-- twelve 30 degree steps, five-second dwell, heading measured as settled
rather than assumed. The half-turn limit is gone: the 271-degree decoy lock it
was added for came from acting on the first frame that said yes, not from
looking too far, so the confidence floor on a dwell is what actually prevents
it. That also makes a banner behind the start heading findable, which is where
seed 1001's return leg kept stranding.

Lettering. Adds a local-contrast stroke path running beside the brightness
path; either may confirm, both feed the same glyph reader. Measured on the
rendered frame under a shade ramp, letters read out of eight: brightness alone
holds the five-letter rescue threshold to 50% shade, both paths to 30%. Full
light still picks brightness, so the rescue does not displace the good path.

Scan ledger, hover, delivery accuracy. An append-only, aggregator-de-duplicated
list of everything decoded, identified or refused, with matches tagged and
refusals keeping their reason, in a right-hand rail. A five-second hover per
DISTINCT payload. WinchDrop now derives the tracking floor from pad size and
camera and raises the drop altitude to it, samples the offset all the way down,
and falls back to the last sighting (converted at the altitude it was taken at,
reported with its age) -- the two causes of `delivery UNMEASURED` on an
otherwise complete run.

sim/record_stage.py promotes the in-flight recorder out of /tmp. --stage is
required: the ungated version of this probe caught the aircraft on the pad and
was one edit from a fourth wrong diagnosis.

Every fix mutation-checked. A review pass then found three more defects the
tests did not (§13.8): a refused leg crashed on its second tick, the centring
timeout measured time-since-phase-entry while reporting time-since-last-seen,
and the new hover opened a window in which one blurred frame could un-make its
own confirmed decode. All three live in transitions, which is where
per-behaviour tests are thinnest.

Not yet demonstrated in a live arena run.

Co-Authored-By: Claude Opus 5 <noreply@anthropic.com>

File: src/aerothon_mission/uav_description/urdf/uav.urdf.xacro (robot description, xacro)
@@ -40,5 +40,11 @@
   <joint name="webcam_pitch_joint" type="revolute">
     <parent link="webcam_servo_base"/><child link="webcam_link"/>
-    <origin xyz="0.045 0 0"/><axis xyz="0 1 0"/><limit lower="-1.570796" upper="0.523599" effort="2" velocity="2"/>
+    <!-- Keep in sync with scripts/materialize_vehicle_model.py: lower limit is
+         -1.65 rad so a -90 deg NADIR command is not sitting on the hard stop. -->
+    <!-- Axis is -Y so that a negative angle pitches the camera DOWN, matching
+         goal.md Q18 and MAVLink DO_MOUNT_CONTROL. See the note in
+         scripts/materialize_vehicle_model.py: with +Y, "-90 deg NADIR" aimed
+         the camera at the sky. Keep the two files in sync. -->
+    <origin xyz="0.045 0 0"/><axis xyz="0 -1 0"/><limit lower="-1.65" upper="0.523599" effort="2" velocity="2"/>
   </joint>
   <link name="webcam_link">

Commit message: Fly the team's real airframe, built from its CAD
The simulator's default vehicle is now the team's quad instead of the
ArduPilot Iris (AEROTHON_AIRFRAME=iris keeps the old one).

- scripts/cad_to_gazebo.py turns the CAD export in "Drone frame/" into
  Gazebo assets: 1.9 M triangles decimated to 78 k, props scaled to 9.45 in,
  the C270 as its own tilting mesh, and airframe.json with the measured
  motor hubs, prop plane, sensor and payload mounts, and the 2.0 kg mass,
  centre of mass and inertia.
- scripts/build_cad_vehicle.py builds the vehicle: ArduPilot quad-X rotors
  at the CAD hubs, thrust for a 2312 980 KV on a 9450 at 4S, LD06 lidar
  (450 pts, 10 Hz, blind to the props) and C270 camera (48.8 deg) at their
  mounts, and the winch hook at the drop mechanism.
- The TF tree (uav.urdf.xacro) and the perception stack's camera FOV follow
  the chosen airframe.
- Gravity hook: the winch pays out past touchdown, and in Gazebo the hook
  lets go when the line goes slack.
- Fixes found flying it: a stiffer camera servo; start marker, target match
  and landing all keep a ground fix instead of holding blind when the
  narrower camera loses the marker at the frame edge; the sweep waits for
  the matched pad's position; the landing starts high enough to lock.

Shipped world on the team airframe: COMPLETED, 14/14 checks, payload
0.13 m from the pad centre, precise landing. Suite: 1054 passed.

Co-Authored-By: Claude Opus 5.5 <noreply@anthropic.com>

File: src/aerothon_mission/uav_description/urdf/uav.urdf.xacro (robot description, xacro)
@@ -1,5 +1,15 @@
 <?xml version="1.0"?>
 <robot xmlns:xacro="http://www.ros.org/wiki/xacro" name="aerothon_iris">
-  <!-- RViz representation of the same official ArduPilot Iris used in Gazebo. -->
+  <!-- The TF tree of the vehicle Gazebo flies, for RViz, slam_toolbox and
+       anything that places a scan or an image in space.
+       airframe:=cad  (default) the team's airframe; mounts measured off its
+                      CAD by scripts/cad_to_gazebo.py (airframe.json) and
+                      used by scripts/build_cad_vehicle.py. Keep in sync.
+       airframe:=iris the ArduPilot Iris variant flown before the CAD arrived.
+       The frames that matter are base_scan (the LD06 / C1 scan origin),
+       webcam_link / camera_optical_frame and winch_link: the geometry of
+       every measurement hangs off them. The visuals are schematic. -->
+  <xacro:arg name="airframe" default="cad"/>
+  <xacro:property name="cad" value="${'$(arg airframe)' == 'cad'}"/>
   <material name="carbon"><color rgba="0.06 0.07 0.08 1"/></material>
   <material name="black"><color rgba="0.015 0.018 0.022 1"/></material>
@@ -9,51 +19,71 @@
   <material name="rplidar_white"><color rgba="0.96 0.97 0.98 1"/></material>
   <material name="orange"><color rgba="1.0 0.42 0.03 1"/></material>
+  <xacro:if value="${cad}">
+    <!-- LD06 on its raised mount on the front plate; C270 pivoting at its
+         own centre; hook under the dropping mechanism. -->
+    <xacro:property name="scan_xyz" value="0.139 -0.002 0.082"/>
+    <xacro:property name="servo_xyz" value="0.163 -0.008 0.008"/>
+    <xacro:property name="pivot_xyz" value="0 0 0"/>
+    <xacro:property name="lens_x" value="0.026"/>
+    <xacro:property name="winch_xyz" value="0 -0.0015 -0.070"/>
+    <xacro:property name="rotor_z" value="0.0706"/>
+    <xacro:property name="rx" value="0.172"/>
+    <xacro:property name="ry" value="0.170"/>
+  </xacro:if>
+  <xacro:unless value="${cad}">
+    <xacro:property name="scan_xyz" value="0 0 0.19"/>
+    <xacro:property name="servo_xyz" value="0.145 0 0.035"/>
+    <xacro:property name="pivot_xyz" value="0.045 0 0"/>
+    <xacro:property name="lens_x" value="0.093"/>
+    <xacro:property name="winch_xyz" value="0 0 -0.10"/>
+    <xacro:property name="rotor_z" value="0.023"/>
+    <xacro:property name="rx" value="0.13"/>
+    <xacro:property name="ry" value="0.21"/>
+  </xacro:unless>
   <link name="base_link">
-    <visual>
-      <geometry><mesh filename="package://ardupilot_gazebo/models/iris_with_standoffs/meshes/iris.dae"/></geometry>
-      <material name="carbon"/>
-    </visual>
-    <collision><geometry><cylinder radius="0.30" length="0.12"/></geometry></collision>
-    <inertial><mass value="1.5"/><inertia ixx="0.029" ixy="0" ixz="0" iyy="0.029" iyz="0" izz="0.055"/></inertial>
+    <xacro:if value="${cad}">
+      <visual><geometry><box size="0.32 0.12 0.10"/></geometry><material name="carbon"/></visual>
+      <collision><geometry><box size="0.32 0.12 0.10"/></geometry></collision>
+      <inertial><mass value="1.87"/><inertia ixx="0.0182" ixy="0" ixz="0" iyy="0.0257" iyz="0" izz="0.0337"/></inertial>
+    </xacro:if>
+    <xacro:unless value="${cad}">
+      <visual>
+        <geometry><mesh filename="package://ardupilot_gazebo/models/iris_with_standoffs/meshes/iris.dae"/></geometry>
+        <material name="carbon"/>
+      </visual>
+      <collision><geometry><cylinder radius="0.30" length="0.12"/></geometry></collision>
+      <inertial><mass value="1.5"/><inertia ixx="0.029" ixy="0" ixz="0" iyy="0.029" iyz="0" izz="0.055"/></inertial>
+    </xacro:unless>
   </link>
-  <xacro:macro name="iris_rotor" params="name x y mesh">
-    <joint name="${name}_fixed" type="fixed"><parent link="base_link"/><child link="${name}"/><origin xyz="${x} ${y} 0.023"/></joint>
-    <link name="${name}"><visual><geometry><mesh filename="package://ardupilot_gazebo/models/iris_with_standoffs/meshes/${mesh}"/></geometry></visual></link>
+  <!-- ArduPilot quad-X order: rotor_0 FR, rotor_1 BL, rotor_2 FL, rotor_3 BR. -->
+  <xacro:macro name="rotor" params="name x y">
+    <joint name="${name}_fixed" type="fixed"><parent link="base_link"/><child link="${name}"/><origin xyz="${x} ${y} ${rotor_z}"/></joint>
+    <link name="${name}"><visual><geometry><cylinder radius="0.12" length="0.004"/></geometry><material name="black"/></visual></link>
   </xacro:macro>
-  <xacro:iris_rotor name="rotor_0" x="0.13" y="-0.22" mesh="iris_prop_ccw.dae"/>
-  <xacro:iris_rotor name="rotor_1" x="-0.13" y="0.20" mesh="iris_prop_ccw.dae"/>
-  <xacro:iris_rotor name="rotor_2" x="0.13" y="0.22" mesh="iris_prop_cw.dae"/>
-  <xacro:iris_rotor name="rotor_3" x="-0.13" y="-0.20" mesh="iris_prop_cw.dae"/>
-  <!-- RPLIDAR C1: top-centre, with a 360-degree unobstructed scan plane. -->
-  <joint name="rplidar_c1_mount" type="fixed"><parent link="base_link"/><child link="base_scan"/><origin xyz="0 0 0.19"/></joint>
+  <xacro:rotor name="rotor_0" x="${rx}" y="${-ry}"/>
+  <xacro:rotor name="rotor_1" x="${-rx}" y="${ry}"/>
+  <xacro:rotor name="rotor_2" x="${rx}" y="${ry}"/>
+  <xacro:rotor name="rotor_3" x="${-rx}" y="${-ry}"/>
+  <!-- The lidar's scan origin. -->
+  <joint name="rplidar_c1_mount" type="fixed"><parent link="base_link"/><child link="base_scan"/><origin xyz="${scan_xyz}"/></joint>
   <link name="base_scan">
-    <visual><origin xyz="0 0 0.018"/><geometry><cylinder radius="0.060" length="0.036"/></geometry><material name="rplidar_white"/></visual>
-    <visual><origin xyz="0 0 0.037"/><geometry><cylinder radius="0.050" length="0.008"/></geometry><material name="rplidar_blue"/></visual>
-    <visual><origin xyz="0 0 0.043"/><geometry><cylinder radius="0.044" length="0.018"/></geometry><material name="black"/></visual>
-    <collision><origin xyz="0 0 0.022"/><geometry><cylinder radius="0.060" length="0.050"/></geometry></collision>
+    <visual><geometry><cylinder radius="0.02" length="0.035"/></geometry><material name="black"/></visual>
   </link>
-  <!-- Front webcam on one pitch servo: 0 rad forward, -1.5708 downward. -->
-  <joint name="webcam_servo_mount" type="fixed"><parent link="base_link"/><child link="webcam_servo_base"/><origin xyz="0.145 0 0.035"/></joint>
-  <link name="webcam_servo_base">
-    <visual><geometry><box size="0.050 0.075 0.055"/></geometry><material name="black"/></visual>
-  </link>
+  <!-- Front camera on one pitch servo: 0 rad forward, -1.5708 downward. -->
+  <joint name="webcam_servo_mount" type="fixed"><parent link="base_link"/><child link="webcam_servo_base"/><origin xyz="${servo_xyz}"/></joint>
+  <link name="webcam_servo_base"/>
   <joint name="webcam_pitch_joint" type="revolute">
     <parent link="webcam_servo_base"/><child link="webcam_link"/>
-    <!-- Keep in sync with scripts/materialize_vehicle_model.py: lower limit is
-         -1.65 rad so a -90 deg NADIR command is not sitting on the hard stop. -->
-    <!-- Axis is -Y so that a negative angle pitches the camera DOWN, matching
-         goal.md Q18 and MAVLink DO_MOUNT_CONTROL. See the note in
-         scripts/materialize_vehicle_model.py: with +Y, "-90 deg NADIR" aimed
-         the camera at the sky. Keep the two files in sync. -->
-    <origin xyz="0.045 0 0"/><axis xyz="0 -1 0"/><limit lower="-1.65" upper="0.523599" effort="2" velocity="2"/>
+    <!-- Keep in sync with the Gazebo model: lower limit -1.65 rad so a -90 deg
+         NADIR command is not on the hard stop, and axis -Y so a NEGATIVE
+         angle pitches DOWN (goal.md Q18, MAVLink DO_MOUNT_CONTROL). -->
+    <origin xyz="${pivot_xyz}"/><axis xyz="0 -1 0"/><limit lower="-1.65" upper="0.523599" effort="2" velocity="2"/>
   </joint>
   <link name="webcam_link">
-    <visual><origin xyz="0.040 0 0"/><geometry><box size="0.080 0.125 0.045"/></geometry><material name="logitech"/></visual>
-    <visual><origin xyz="0.087 0 0" rpy="0 1.570796 0"/><geometry><cylinder radius="0.012" length="0.010"/></geometry><material name="lens"/></visual>
-    <collision><origin xyz="0.040 0 0"/><geometry><box size="0.080 0.125 0.045"/></geometry></collision>
+    <visual><geometry><box size="0.030 0.071 0.030"/></geometry><material name="logitech"/></visual>
   </link>
-  <joint name="camera_optical_joint" type="fixed"><parent link="webcam_link"/><child link="camera_optical_frame"/><origin xyz="0.093 0 0" rpy="-1.570796 0 -1.570796"/></joint>
+  <joint name="camera_optical_joint" type="fixed"><parent link="webcam_link"/><child link="camera_optical_frame"/><origin xyz="${lens_x} 0 0" rpy="-1.570796 0 -1.570796"/></joint>
   <link name="camera_optical_frame"/>
-  <joint name="winch_joint" type="fixed"><parent link="base_link"/><child link="winch_link"/><origin xyz="0 0 -0.10"/></joint>
+  <joint name="winch_joint" type="fixed"><parent link="base_link"/><child link="winch_link"/><origin xyz="${winch_xyz}"/></joint>
   <link name="winch_link"><visual><geometry><cylinder radius="0.03" length="0.05"/></geometry><material name="orange"/></visual></link>
 </robot>
